File: ruler_pcb.kicad_pcb (KiCad board)
At the start: 2 copper layers, 306.3 x 38.1 mm, 71 parts

Commit message: Updated schematic page info and size
Parts:
- moved G*** 2.54 mm to (289.6, 72.4)
- moved REF** 2.54 mm to (139.2, 63.8)
- moved REF** 2.54 mm to (139.2, 69.8)
- moved REF** 2.54 mm to (139.2, 75.9)
- moved REF** 2.54 mm to (139.2, 82.3)
- moved REF** 2.54 mm to (163.8, 79.8)
- moved REF** 2.54 mm to (155.4, 79.8)
- moved REF** 2.54 mm to (179.3, 82.0)
- moved REF** 2.54 mm to (171.7, 81.5)
- moved REF** 2.54 mm to (171.7, 73.7)
- moved REF** 2.54 mm to (179.3, 75.7)
- moved REF** 2.54 mm to (179.3, 68.3)
- moved REF** 2.54 mm to (171.7, 65.3)
- moved REF** 2.54 mm to (187.2, 69.3)
- moved REF** 2.54 mm to (53.3, 78.7)
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Other:
- board text added: "rev 1.0 Robin S. Yang"
- board text removed: "rev 1.0 Robin Yang"
