File: ruler_pcb.kicad_pcb (KiCad board)
At the start: 2 copper layers, 306.3 x 38.1 mm, 71 parts

Commit message: vt-var-br
Parts:
- removed the G*** at (19.7, 72.4)
- removed the G*** at (289.6, 72.4)
- added G***: LOGO, ruler_specific:VT_SHIELD_SMALLER, B.Cu at (90.7, 59.4)
- added G***: LOGO, ruler_specific:VT_NEW_TEXT_ONLY, F.Cu at (277.6, 72.4)
- added G***: LOGO, ruler_specific:VT_NEW_VT, F.Cu at (288.5, 72.4)
- added G***: LOGO, ruler_specific:VT_OLD_VERTICAL, B.Cu at (294.6, 71.9)
Other:
- board text added: "For Personal Use Only Designed By RY"
- board text removed: "1.2 1.8 3.0 5.6 10.6 20.6 40.6 60.6"
- board text removed: "120V 240V 480V 1KV 2KV 4KV 8KV 12KV"
- board text removed: "CREEPAGE(MM)"
- board text removed: "PCB RULER"
- board text removed: "rev 1.0 Robin S. Yang"
